Commit message: 2026 06.23 09：30

File: wvcsc_sensor_kit_launch/wvcsc_sensor_kit_description/urdf/sensors.xacro (robot description, xacro)
@@ -2,14 +2,61 @@
 <robot name="vehicle" xmlns:xacro="http://ros.org/wiki/xacro">
   <xacro:arg name="config_dir" default="$(find wvcsc_sensor_kit_description)/config"/>
-  <xacro:property name="calibration" value="${xacro.load_yaml('$(arg config_dir)/sensors_calibration.yaml')}"/>
-  <xacro:include filename="sensor_kit.xacro"/>
+  <xacro:property name="sensors_calibration" value="${xacro.load_yaml('$(arg config_dir)/sensors_calibration.yaml')}"/>
+  <xacro:macro name="sensor_kit_macro" params="parent x y z roll pitch yaw">
+    <xacro:property name="sensor_kit_calibration" value="${xacro.load_yaml('$(arg config_dir)/sensor_kit_calibration.yaml')}"/>
+    <xacro:property name="sensor_kit_base_link" value="sensor_kit_base_link"/>
+    <joint name="${sensor_kit_base_link}_joint" type="fixed">
+      <origin xyz="${x} ${y} ${z}" rpy="${roll} ${pitch} ${yaw}"/>
+      <parent link="${parent}"/>
+      <child link="${sensor_kit_base_link}"/>
+    </joint>
+    <link name="${sensor_kit_base_link}"/>
+    <joint name="laser_joint" type="fixed">
+      <origin
+        xyz="${sensor_kit_calibration['sensor_kit_base_link']['laser']['x']} ${sensor_kit_calibration['sensor_kit_base_link']['laser']['y']} ${sensor_kit_calibration['sensor_kit_base_link']['laser']['z']}"
+        rpy="${sensor_kit_calibration['sensor_kit_base_link']['laser']['roll']} ${sensor_kit_calibration['sensor_kit_base_link']['laser']['pitch']} ${sensor_kit_calibration['sensor_kit_base_link']['laser']['yaw']}"
+      />
+      <parent link="${sensor_kit_base_link}"/>
+      <child link="laser"/>
+    </joint>
+    <link name="laser">
+      <visual>
+        <origin xyz="0 0 0" rpy="0 0 0"/>
+        <geometry>
+          <cylinder radius="0.08" length="0.15"/>
+        </geometry>
+        <material name="laser_gray">
+          <color rgba="0.5 0.5 0.5 1"/>
+        </material>
+      </visual>
+    </link>
+    <joint name="gyro_link_joint" type="fixed">
+      <origin
+        xyz="${sensor_kit_calibration['sensor_kit_base_link']['gyro_link']['x']} ${sensor_kit_calibration['sensor_kit_base_link']['gyro_link']['y']} ${sensor_kit_calibration['sensor_kit_base_link']['gyro_link']['z']}"
+        rpy="${sensor_kit_calibration['sensor_kit_base_link']['gyro_link']['roll']} ${sensor_kit_calibration['sensor_kit_base_link']['gyro_link']['pitch']} ${sensor_kit_calibration['sensor_kit_base_link']['gyro_link']['yaw']}"
+      />
+      <parent link="${sensor_kit_base_link}"/>
+      <child link="gyro_link"/>
+    </joint>
+    <link name="gyro_link">
+      <visual>
+        <origin xyz="0 0 0" rpy="0 0 0"/>
+        <geometry>
+          <box size="0.1 0.1 0.001"/>
+        </geometry>
+        <material name="gyro_gray">
+          <color rgba="0.5 0.5 0.5 1"/>
+        </material>
+      </visual>
+    </link>
+  </xacro:macro>
   <xacro:sensor_kit_macro
     parent="base_link"
-    x="${calibration['base_link']['sensor_kit_base_link']['x']}"
-    y="${calibration['base_link']['sensor_kit_base_link']['y']}"
-    z="${calibration['base_link']['sensor_kit_base_link']['z']}"
-    roll="${calibration['base_link']['sensor_kit_base_link']['roll']}"
-    pitch="${calibration['base_link']['sensor_kit_base_link']['pitch']}"
-    yaw="${calibration['base_link']['sensor_kit_base_link']['yaw']}"
+    x="${sensors_calibration['base_link']['sensor_kit_base_link']['x']}"
+    y="${sensors_calibration['base_link']['sensor_kit_base_link']['y']}"
+    z="${sensors_calibration['base_link']['sensor_kit_base_link']['z']}"
+    roll="${sensors_calibration['base_link']['sensor_kit_base_link']['roll']}"
+    pitch="${sensors_calibration['base_link']['sensor_kit_base_link']['pitch']}"
+    yaw="${sensors_calibration['base_link']['sensor_kit_base_link']['yaw']}"
   />
 </robot>

File: wvcsc_vehicle_launch/wvcsc_vehicle_description/urdf/vehicle.xacro (robot description, xacro)
@@ -1,16 +1,76 @@
 <?xml version="1.0"?>
-<robot xmlns:xacro="http://ros.org/wiki/xacro">
+<robot name="wvcsc_vehicle" xmlns:xacro="http://ros.org/wiki/xacro">
+  <xacro:arg name="vehicle_model" default="wvcsc_vehicle"/>
+  <xacro:arg name="sensor_model" default="wvcsc_sensor_kit"/>
+  <xacro:arg name="config_dir" default="$(find wvcsc_sensor_kit_description)/config"/>
+  <!-- Keep the previous full-vehicle behavior in one vehicle description file. -->
   <xacro:property name="vehicle_info" value="${xacro.load_yaml('$(find wvcsc_vehicle_description)/config/vehicle_info.param.yaml')}"/>
-  <xacro:property name="params" value="${vehicle_info['/**']['ros__parameters']}"/>
-  <xacro:include filename="$(find wvcsc_vehicle_description)/urdf/wvcsc_vehicle_base.xacro"/>
-  <xacro:wvcsc_vehicle_base_macro
-    base_length="${params['vehicle_length']}"
-    base_width="0.80"
-    base_height="${params['vehicle_height']}"
-    base_link_to_footprint_z="0.66"
-    wheel_radius="${params['wheel_radius']}"
-    wheel_width="${params['wheel_width']}"
-    wheel_x="${params['wheel_base'] / 2.0}"
-    wheel_y="${params['wheel_tread'] / 2.0}"
+  <xacro:property name="vehicle_params" value="${vehicle_info['/**']['ros__parameters']}"/>
+  <xacro:property name="base_width" value="0.80"/>
+  <xacro:property name="base_link_to_footprint_z" value="0.66"/>
+  <material name="white">
+    <color rgba="1 1 1 1"/>
+  </material>
+  <material name="black">
+    <color rgba="0 0 0 1"/>
+  </material>
+  <link name="base_footprint">
+    <visual>
+      <origin xyz="0 0 0" rpy="0 0 0"/>
+      <geometry>
+        <box size="0.1 0.1 0.001"/>
+      </geometry>
+    </visual>
+  </link>
+  <joint name="base_footprint_joint" type="fixed">
+    <parent link="base_link"/>
+    <child link="base_footprint"/>
+    <origin xyz="0 0 ${-base_link_to_footprint_z}" rpy="0 0 0"/>
+  </joint>
+  <link name="base_link">
+    <visual>
+      <origin xyz="0 0 0" rpy="0 0 0"/>
+      <geometry>
+        <box size="${vehicle_params['vehicle_length']} ${base_width} ${vehicle_params['vehicle_height']}"/>
+      </geometry>
+      <material name="white"/>
+    </visual>
+  </link>
+  <xacro:macro name="wvcsc_wheel_macro" params="wheel_name x y">
+    <joint name="${wheel_name}_joint" type="continuous">
+      <origin xyz="${x} ${y} ${-vehicle_params['vehicle_height'] / 2.0}" rpy="1.57 0 0"/>
+      <parent link="base_link"/>
+      <child link="${wheel_name}_link"/>
+      <axis xyz="0 1 0"/>
+    </joint>
+    <link name="${wheel_name}_link">
+      <visual>
+        <origin xyz="0 0 0" rpy="0 0 0"/>
+        <geometry>
+          <cylinder radius="${vehicle_params['wheel_radius']}" length="${vehicle_params['wheel_width']}"/>
+        </geometry>
+        <material name="black"/>
+      </visual>
+    </link>
+  </xacro:macro>
+  <xacro:wvcsc_wheel_macro
+    wheel_name="left_front"
+    x="${vehicle_params['wheel_base'] / 2.0}"
+    y="${vehicle_params['wheel_tread'] / 2.0}"
+  />
+  <xacro:wvcsc_wheel_macro
+    wheel_name="right_front"
+    x="${vehicle_params['wheel_base'] / 2.0}"
+    y="${-vehicle_params['wheel_tread'] / 2.0}"
+  />
+  <xacro:wvcsc_wheel_macro
+    wheel_name="left_wheel"
+    x="${-vehicle_params['wheel_base'] / 2.0}"
+    y="${vehicle_params['wheel_tread'] / 2.0}"
+  />
+  <xacro:wvcsc_wheel_macro
+    wheel_name="right_wheel"
+    x="${-vehicle_params['wheel_base'] / 2.0}"
+    y="${-vehicle_params['wheel_tread'] / 2.0}"
   />
 </robot>
